File: dimmer/dimmer.kicad_sch (KiCad schematic)
At the start: 11 parts, among them U1 NE555P

Commit message: final course adjustments
Other:
- title: Smart Lighting: Dimmer -> Smart Lighting: Dimmer Control Circuit
- moved on the sheet: D3, D4, R1, R3
Changed lines of the file:
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@@
 	(paper "USLetter")
 	(title_block
-		(title "Smart Lighting: Dimmer")
+		(title "Smart Lighting: Dimmer Control Circuit")
 		(date "May 27, 2026")
 		(rev "A")
@@
 	)
 	(junction
+		(at 133.35 111.76)
+		(diameter 0)
+		(color 0 0 0 0)
+	)
+	(junction
 		(at 114.3 81.28)
 		(diameter 0)
@@
 	)
 	(junction
-		(at 162.56 111.76)
-		(diameter 0)
-		(color 0 0 0 0)
-	)
-	(junction
 		(at 101.6 73.66)
 		(diameter 0)
@@
 	)
 	(junction
-		(at 133.35 111.76)
+		(at 152.4 111.76)
 		(diameter 0)
 		(color 0 0 0 0)
@@
 	(wire
 		(pts
-			(xy 143.51 76.2) (xy 162.56 76.2)
+			(xy 143.51 76.2) (xy 152.4 76.2)
 		)
 		(stroke
@@
 	(wire
 		(pts
-			(xy 187.96 111.76) (xy 187.96 104.14)
+			(xy 168.91 111.76) (xy 168.91 104.14)
 		)
 		(stroke
@@
 	(wire
 		(pts
-			(xy 187.96 91.44) (xy 187.96 96.52)
+			(xy 168.91 91.44) (xy 168.91 96.52)
 		)
 		(stroke
@@
 	(wire
 		(pts
-			(xy 187.96 40.64) (xy 187.96 83.82)
-		)
-		(stroke
-			(width 0)
-			(type default)
-		)
-	)
-	(wire
-		(pts
-			(xy 162.56 111.76) (xy 187.96 111.76)
+			(xy 168.91 40.64) (xy 168.91 83.82)
+		)
+		(stroke
+			(width 0)
+			(type default)
+		)
+	)
+	(wire
+		(pts
+			(xy 152.4 111.76) (xy 168.91 111.76)
 		)
 		(stroke
@@
 	(wire
 		(pts
-			(xy 135.89 40.64) (xy 187.96 40.64)
-		)
-		(stroke
-			(width 0)
-			(type default)
-		)
-	)
-	(wire
-		(pts
-			(xy 162.56 91.44) (xy 162.56 96.52)
-		)
-		(stroke
-			(width 0)
-			(type default)
-		)
-	)
-	(wire
-		(pts
-			(xy 162.56 111.76) (xy 162.56 104.14)
-		)
-		(stroke
-			(width 0)
-			(type default)
-		)
-	)
-	(wire
-		(pts
-			(xy 162.56 76.2) (xy 162.56 83.82)
+			(xy 135.89 40.64) (xy 168.91 40.64)
+		)
+		(stroke
+			(width 0)
+			(type default)
+		)
+	)
+	(wire
+		(pts
+			(xy 152.4 91.44) (xy 152.4 96.52)
+		)
+		(stroke
+			(width 0)
+			(type default)
+		)
+	)
+	(wire
+		(pts
+			(xy 152.4 111.76) (xy 152.4 104.14)
+		)
+		(stroke
+			(width 0)
+			(type default)
+		)
+	)
+	(wire
+		(pts
+			(xy 152.4 76.2) (xy 152.4 83.82)
 		)
 		(stroke
@@
 	(wire
 		(pts
-			(xy 133.35 111.76) (xy 162.56 111.76)
+			(xy 133.35 111.76) (xy 152.4 111.76)
 		)
 		(stroke
@@
 	(symbol
 		(lib_id "Device:R")
-		(at 187.96 87.63 0)
+		(at 168.91 87.63 0)
 		(unit 1)
 		(body_style 1)
@@
 		(fields_autoplaced yes)
 		(property "Reference" "R3"
-			(at 190.5 86.3599 0)
+			(at 171.45 86.3599 0)
 			(show_name no)
 			(do_not_autoplace no)
@@
 		)
 		(property "Value" "200"
-			(at 190.5 88.8999 0)
+			(at 171.45 88.8999 0)
 			(show_name no)
 			(do_not_autoplace no)
@@
 		)
 		(property "Footprint" "Resistor_THT:R_Axial_DIN0207_L6.3mm_D2.5mm_P10.16mm_Horizontal"
-			(at 186.182 87.63 90)
+			(at 167.132 87.63 90)
 			(hide yes)
 			(show_name no)
@@
 		)
 		(property "Datasheet" ""
-			(at 187.96 87.63 0)
+			(at 168.91 87.63 0)
 			(hide yes)
 			(show_name no)
@@
 		)
 		(property "Description" "Resistor"
-			(at 187.96 87.63 0)
+			(at 168.91 87.63 0)
 			(hide yes)
 			(show_name no)
@@
 	(symbol
 		(lib_id "Device:LED")
-		(at 187.96 100.33 90)
+		(at 168.91 100.33 90)
 		(unit 1)
 		(body_style 1)
@@
 		(fields_autoplaced yes)
 		(property "Reference" "D4"
-			(at 191.77 100.6474 90)
+			(at 172.72 100.6474 90)
 			(show_name no)
 			(do_not_autoplace no)
@@
 		)
 		(property "Value" "LED"
-			(at 191.77 103.1874 90)
+			(at 172.72 103.1874 90)
 			(show_name no)
 			(do_not_autoplace no)
@@
 		)
 		(property "Footprint" "LED_THT:LED_D5.0mm_Clear"
-			(at 187.96 100.33 0)
+			(at 168.91 100.33 0)
 			(hide yes)
 			(show_name no)
@@
 		)
 		(property "Datasheet" ""
-			(at 187.96 100.33 0)
+			(at 168.91 100.33 0)
 			(hide yes)
 			(show_name no)
@@
 		)
 		(property "Description" "Light emitting diode"
-			(at 187.96 100.33 0)
+			(at 168.91 100.33 0)
 			(hide yes)
 			(show_name no)
@@
 		)
 		(property "Sim.Pins" "1=K 2=A"
-			(at 187.96 100.33 0)
+			(at 168.91 100.33 0)
 			(hide yes)
 			(show_name no)
@@
 	(symbol
 		(lib_id "Device:LED")
-		(at 162.56 100.33 90)
+		(at 152.4 100.33 90)
 		(unit 1)
 		(body_style 1)
@@
 		(fields_autoplaced yes)
 		(property "Reference" "D3"
-			(at 166.37 100.6474 90)
+			(at 156.21 100.6474 90)
 			(show_name no)
 			(do_not_autoplace no)
@@
 		)
 		(property "Value" "LED"
-			(at 166.37 103.1874 90)
+			(at 156.21 103.1874 90)
 			(show_name no)
 			(do_not_autoplace no)
@@
 		)
 		(property "Footprint" "LED_THT:LED_D5.0mm_Clear"
-			(at 162.56 100.33 0)
+			(at 152.4 100.33 0)
 			(hide yes)
 			(show_name no)
@@
 		)
 		(property "Datasheet" ""
-			(at 162.56 100.33 0)
+			(at 152.4 100.33 0)
 			(hide yes)
 			(show_name no)
@@
 		)
 		(property "Description" "Light emitting diode"
-			(at 162.56 100.33 0)
+			(at 152.4 100.33 0)
 			(hide yes)
 			(show_name no)
@@
 		)
 		(property "Sim.Pins" "1=K 2=A"
-			(at 162.56 100.33 0)
+			(at 152.4 100.33 0)
 			(hide yes)
 			(show_name no)
@@
 	(symbol
 		(lib_id "Device:R")
-		(at 162.56 87.63 0)
+		(at 152.4 87.63 0)
 		(unit 1)
 		(body_style 1)
@@
 		(fields_autoplaced yes)
 		(property "Reference" "R1"
-			(at 165.1 86.3599 0)
+			(at 154.94 86.3599 0)
 			(show_name no)
 			(do_not_autoplace no)
@@
 		)
 		(property "Value" "200"
-			(at 165.1 88.8999 0)
+			(at 154.94 88.8999 0)
 			(show_name no)
 			(do_not_autoplace no)
@@
 		)
 		(property "Footprint" "Resistor_THT:R_Axial_DIN0207_L6.3mm_D2.5mm_P10.16mm_Horizontal"
-			(at 160.782 87.63 90)
+			(at 150.622 87.63 90)
 			(hide yes)
 			(show_name no)
@@
 		)
 		(property "Datasheet" ""
-			(at 162.56 87.63 0)
+			(at 152.4 87.63 0)
 			(hide yes)
 			(show_name no)
@@
 		)
 		(property "Description" "Resistor"
-			(at 162.56 87.63 0)
-			(hide yes)
-			(show_name no)
+			(at 152.4 87.63 0)
+			(hide yes)
+			(show_name no)
