File: ledcomms/ledcomms.kicad_sch (KiCad schematic)
At the start: 16 parts, among them J1 Power, J2 Digital/PWM, J3 Analog, J4 Digital/PWM, U1 LM741, U2 LM393

Commit message: final course adjustments
Parts:
- R1: now not fitted
- R2: value 1.5M -> 1k
Other:
- moved on the sheet: D1, D2, D3, J2, J3, J4, R2, R3, R4, R5, R6, R7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
